File: hardware/dji-fcc.kicad_pcb (KiCad board)
At the start: 2 copper layers, 76 x 34 mm, 70 parts, among them J1 USB-C REMOTE, J2 USB-C CHARGE, J3 BATTERY 1S LiPo (+ on pin 1), Q1 FS8205A, U1 ESP32-S3-MINI-1-N8, U2 AP2112K-3.3, U3 TP4056, U4 DW01A, U5 MT3608, U6 TPS2553DBVR, U7 USBLC6-2SC6

Commit message: Flash and update over USB-C: FSUSB42 data switch between J1/J2, charge status on ESP, wider board
Parts:
- removed D2: RED, LED_SMD:LED_0603_1608Metric
- removed D3: GREEN, LED_SMD:LED_0603_1608Metric
- removed R5, R6: 1k, Resistor_SMD:R_0603_1608Metric
- added C15: 100nF, Capacitor_SMD:C_0603_1608Metric, F.Cu at (44.6, 26.6)
- added U8: FSUSB42MUX, Package_SO:MSOP-10_3x3mm_P0.5mm, F.Cu at (49.4, 23.4)
- added U9: USBLC6-2SC6, Package_TO_SOT_SMD:SOT-23-6, F.Cu at (68.2, 23.4)
- moved TP7 22.8 mm to (7.00, 28.2)
- moved TP8 20.5 mm to (7.00, 25.4)
- moved C1 4.00 mm to (53.0, 7.80)
- moved C4 4.00 mm to (64.0, 8.50)
- moved C5 4.00 mm to (52.5, 11.0)
- moved C6 4.00 mm to (67.5, 11.5)
- moved C7 4.00 mm to (64.0, 21.5)
- moved C8 4.00 mm to (62.5, 30.0)
- moved D1 4.00 mm to (72.5, 9.10)
- moved D6 4.00 mm to (67.0, 2.20)
- moved D7 4.00 mm to (71.0, 2.20)
- moved D8 4.00 mm to (75.0, 2.20)
- moved FID2 4.00 mm to (77.5, 8.00)
- moved FID3 4.00 mm to (78.0, 25.0)
- moved H1 4.00 mm to (77.0, 31.0)
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Connections:
- J2 pad A6: unconnected-(J2-D+-PadA6) -> USB2_DP_C
- J2 pad A7: unconnected-(J2-D--PadA7) -> USB2_DN_C
- J2 pad B6: unconnected-(J2-D+-PadB6) -> USB2_DP_C
- J2 pad B7: unconnected-(J2-D--PadB7) -> USB2_DN_C
- U1 pad 25: unconnected-(U1-IO21-Pad25) -> VCHG_SENSE
- U1 pad 34: VCHG_SENSE -> STDBY
- U1 pad 35: unconnected-(U1-IO39-Pad35) -> CHRG
- U7 pad 4: USB_DN -> USB_DN_J1
- U7 pad 6: USB_DP -> USB_DP_J1
Routing:
- net USB_DP_J1: track 0.00 -> 27.0 mm, vias 0 -> 2
- net USB_DN_J1: track 0.00 -> 26.6 mm, vias 0 -> 2
- net GND: track 172.3 -> 197.9 mm, vias 47 -> 48
- net USB2_DN_C: track 0.00 -> 20.8 mm, vias 0 -> 2
- net USB2_DP: track 0.00 -> 20.5 mm
- net USB2_DN: track 0.00 -> 19.0 mm
- net +3V3: track 146.8 -> 128.1 mm
- net VBAT: track 156.2 -> 172.5 mm, vias 6 -> 5
- net VCHG_SENSE: track 10.3 -> 24.7 mm, vias 2 -> 4
- net ESP_EN: track 37.5 -> 51.3 mm
- net USB2_DP_C: track 0.00 -> 12.2 mm
- net STDBY: track 19.3 -> 30.0 mm
- net USB_DP_C: track 35.1 -> 24.4 mm
- net DONE_A: track 10.6 -> 0.00 mm, vias 2 -> 0
- net IO0: track 30.5 -> 39.7 mm
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Other:
- board size 76 x 34 mm -> 80 x 34 mm
