File: hardware/dji-fcc.kicad_sch (KiCad schematic)
At the start: 70 parts, among them J1 USB-C REMOTE, J2 USB-C CHARGE, J3 BATTERY 1S LiPo (+ on pin 1), Q1 FS8205A, U1 ESP32-S3-MINI-1-N8, U2 AP2112K-3.3, U3 TP4056, U4 DW01A, U5 MT3608, U6 TPS2553DBVR, U7 USBLC6-2SC6

Commit message: Flash and update over USB-C: FSUSB42 data switch between J1/J2, charge status on ESP, wider board
Parts:
- removed D2: RED, LED_SMD:LED_0603_1608Metric, symbol Device:LED
- removed D3: GREEN, LED_SMD:LED_0603_1608Metric, symbol Device:LED
- removed R5, R6: 1k, Resistor_SMD:R_0603_1608Metric, symbol Device:R
- added C15: 100nF, Capacitor_SMD:C_0603_1608Metric, symbol Device:C
- added U8: FSUSB42MUX, Package_SO:MSOP-10_3x3mm_P0.5mm, symbol Interface_USB:FSUSB42MUX
- added U9: USBLC6-2SC6, Package_TO_SOT_SMD:SOT-23-6, symbol Power_Protection:USBLC6-2SC6
Connections:
- net +3V3: now also C15.1, U8.1 (VCC)
- net CHRG: now also U1.35 (IO39)
- net GND: now also C15.2, U8.10 (~{OE}), U8.5 (GND), U9.2 (GND)
- net STDBY: now also U1.34 (IO38)
- net USB_DN: now also U8.4 (D-); no longer U7.4 (I/O2)
- net USB_DP: now also U8.3 (D+); no longer U7.6 (I/O1)
- net VBUS_CHG: now also U9.5 (VBUS)
- net VCHG_SENSE: now also U1.25 (IO21), U8.2 (SEL); no longer U1.34 (IO38)
- net USB2_DP_C: now reaches J2.A6 (D+)
- net USB2_DP_C: now also J2.B6 (D+), U9.1 (I/O1)
- net USB2_DN_C: now reaches J2.A7 (D-)
- net USB2_DN_C: now also J2.B7 (D-), U9.3 (I/O2)
- new net USB2_DN: U8.8 (HSD2-), U9.4 (I/O2)
- new net USB2_DP: U8.9 (HSD2+), U9.6 (I/O1)
- new net USB_DN_J1: U7.4 (I/O2), U8.6 (HSD1-)
- new net USB_DP_J1: U7.6 (I/O1), U8.7 (HSD1+)
- no-connect marks 35 -> 29
Other:
- note added: "USB data switch (U8): J2 plugged into a computer -> ESP on J2, else ESP on J1"
